File: led.kicad_sch (KiCad schematic)
At the start: 2 parts

Commit message: Final
Parts:
- added BT1: Battery, symbol Device:Battery
Connections:
- net at R1.2: now also BT1.1 (+)
- net at D1.1 (K): now also BT1.2 (-)
Changed lines of the file:
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@@
 (kicad_sch (version 20230121) (generator eeschema)
   (paper "A4")
+  (wire (pts (xy 170.18 88.9) (xy 161.925 88.9))
+    (stroke (width 0) (type default))
+  )
+  (wire (pts (xy 170.18 90.17) (xy 170.18 88.9))
+    (stroke (width 0) (type default))
+  )
+  (wire (pts (xy 137.16 100.33) (xy 137.16 88.9))
+    (stroke (width 0) (type default))
+  )
+  (wire (pts (xy 137.16 88.9) (xy 141.605 88.9))
+    (stroke (width 0) (type default))
+  )
+  (wire (pts (xy 170.18 100.33) (xy 137.16 100.33))
+    (stroke (width 0) (type default))
+  )
   (wire (pts (xy 149.225 88.9) (xy 154.305 88.9))
     (stroke (width 0) (type default))
@@
         )
       )
+    )
+  )
+  (symbol (lib_id "Device:Battery") (at 170.18 95.25 0) (unit 1)
+    (in_bom yes) (on_board yes) (dnp no) (fields_autoplaced)
+    (property "Reference" "BT1" (at 173.99 94.234 0)
+      (effects (font (size 1.27 1.27)) (justify left))
+    )
+    (property "Value" "Battery" (at 173.99 96.774 0)
+      (effects (font (size 1.27 1.27)) (justify left))
+    )
+    (property "Footprint" "" (at 170.18 93.726 90)
+      (effects (font (size 1.27 1.27)) hide)
+    )
+    (property "Datasheet" "~" (at 170.18 93.726 90)
+      (effects (font (size 1.27 1.27)) hide)
+    )
+    (pin "1")
+    (pin "2")
+    (instances
+      (project "led"
+        (path "/814b1cca-5fed-4f5a-ab32-23d28f275249"
+          (reference "BT1") (unit 1)
+        )
+      )
